Commit message: movimiento omnidirecciona

File: src/tadeocar_description/urdf/tadeocar_tf.urdf (robot description, URDF)
Before this commit: robot tadeocar_v1, 5 links, 4 joints
Links:
- removed link camera_link
- removed link imu_link
- removed link lidar_link
- added link base_scan
Joints:
- removed joint camera_joint
- removed joint imu_joint
- joint lidar_joint: child lidar_link -> base_scan; origin xyz=0.6 0 0.4 rpy=0 0 0 -> xyz=0 0 0.30 rpy=0 0 0

Commit message: movimiento omnidireccional left OK

File: src/tadeocar_description/urdf/tadeocar_tf.urdf (robot description, URDF)
Before this commit: robot tadeocar_v1, 3 links, 2 joints
Joints:
- joint lidar_joint: origin xyz=0 0 0.30 rpy=0 0 0 -> xyz=0.55 0 0.39 rpy=0 0 0
