Commit message: camera estereo

File: src/tadeocar_description/urdf/tadeocar_control.urdf.xacro (robot description, xacro)
@@ -66,7 +66,7 @@
   <link name="stereo_camera_base">
     <inertial>
-      <mass value="0.1"/>
-      <origin xyz="0 0 0" rpy="0 0 0"/>
-      <inertia ixx="0.0001" ixy="0.0" ixz="0.0" iyy="0.0001" iyz="0.0" izz="0.0001"/>
+      <mass value="0.5"/>
+      <origin xyz="0 0 0" rpy="0 0 0"/>
+      <inertia ixx="0.001" ixy="0.0" ixz="0.0" iyy="0.001" iyz="0.0" izz="0.001"/>
     </inertial>
     <visual>
@@ -79,10 +79,5 @@
       </material>
     </visual>
-    <collision>
-      <origin xyz="0 0 0" rpy="0 0 1.5708"/>
-      <geometry>
-        <box size="0.15 0.05 0.03"/>
-      </geometry>
-    </collision>
+    <!-- Collision removed - cameras are sensors only -->
   </link>
   <joint name="stereo_camera_base_joint" type="fixed">
@@ -94,7 +89,7 @@
   <link name="camera_left">
     <inertial>
-      <mass value="0.05"/>
-      <origin xyz="0 0 0" rpy="0 0 0"/>
-      <inertia ixx="0.00001" ixy="0.0" ixz="0.0" iyy="0.00001" iyz="0.0" izz="0.00001"/>
+      <mass value="0.2"/>
+      <origin xyz="0 0 0" rpy="0 0 0"/>
+      <inertia ixx="0.0001" ixy="0.0" ixz="0.0" iyy="0.0001" iyz="0.0" izz="0.0001"/>
     </inertial>
     <visual>
@@ -107,10 +102,5 @@
       </material>
     </visual>
-    <collision>
-      <origin xyz="0 0 0" rpy="0 1.5708 0"/>
-      <geometry>
-        <cylinder radius="0.01" length="0.01"/>
-      </geometry>
-    </collision>
+    <!-- Collision removed - cameras are sensors only -->
   </link>
   <joint name="camera_left_joint" type="fixed">
@@ -122,7 +112,7 @@
   <link name="camera_right">
     <inertial>
-      <mass value="0.05"/>
-      <origin xyz="0 0 0" rpy="0 0 0"/>
-      <inertia ixx="0.00001" ixy="0.0" ixz="0.0" iyy="0.00001" iyz="0.0" izz="0.00001"/>
+      <mass value="0.2"/>
+      <origin xyz="0 0 0" rpy="0 0 0"/>
+      <inertia ixx="0.0001" ixy="0.0" ixz="0.0" iyy="0.0001" iyz="0.0" izz="0.0001"/>
     </inertial>
     <visual>
@@ -135,10 +125,5 @@
       </material>
     </visual>
-    <collision>
-      <origin xyz="0 0 0" rpy="0 1.5708 0"/>
-      <geometry>
-        <cylinder radius="0.01" length="0.01"/>
-      </geometry>
-    </collision>
+    <!-- Collision removed - cameras are sensors only -->
   </link>
   <joint name="camera_right_joint" type="fixed">
@@ -334,18 +319,17 @@
     </plugin>
   </gazebo>
-  <!-- Gazebo properties for stereo camera base -->
+  <!-- Gazebo properties for cameras - removed kinematic flag to fix physics issues -->
+  <!-- Camera links are now properly fixed to base_link via joints -->
   <gazebo reference="stereo_camera_base">
-    <gravity>false</gravity>
-    <kinematic>true</kinematic>
-  </gazebo>
-  <!-- Gazebo properties for left camera -->
+    <mu1>0.2</mu1>
+    <mu2>0.2</mu2>
+  </gazebo>
   <gazebo reference="camera_left">
-    <gravity>false</gravity>
-    <kinematic>true</kinematic>
-  </gazebo>
-  <!-- Gazebo properties for right camera -->
+    <mu1>0.2</mu1>
+    <mu2>0.2</mu2>
+  </gazebo>
   <gazebo reference="camera_right">
-    <gravity>false</gravity>
-    <kinematic>true</kinematic>
+    <mu1>0.2</mu1>
+    <mu2>0.2</mu2>
   </gazebo>
   <!-- Gazebo plugin for left camera -->
