Commit message: migration gazebo classic to ignition gazebo, slamtolbox, nav2

File: src/tadeocar_description/urdf/tadeocar.urdf (robot description, URDF)
Before this commit: robot tadeocar, 17 links, 16 joints
Links:
- link base_link: geometry visual mesh 
- link base_scan: geometry visual cylinder length=0.030 radius=0.035
- link camera_left: geometry visual cylinder length=0.01 radius=0.01
- link camera_right: geometry visual cylinder length=0.01 radius=0.01
- link chasis_link: geometry visual mesh 
- link front_left_steering_link: geometry visual mesh 
- link front_left_wheel_link: geometry visual mesh 
- link front_right_steering_link: geometry visual mesh 
- link front_right_wheel_link: geometry visual mesh 
- link rear_left_steering_link: geometry visual mesh 
- link rear_left_wheel_link: geometry visual mesh 
- link rear_right_steering_link: geometry visual mesh 
- link rear_right_wheel_link: geometry visual mesh 
- link stereo_camera_base: geometry visual box size=0.15 0.05 0.03

Commit message: liks visuales

File: src/tadeocar_description/urdf/tadeocar.urdf (robot description, URDF)
Before this commit: robot tadeocar, 17 links, 16 joints
Links:
- link base_link: geometry visual mesh filename=package://tadeocar_description/models/tadeocar_v1/meshes/ch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 scale=1 1 1
- link chasis_link: geometry visual mesh filename=package://tadeocar_description/models/tadeocar_v1/meshes/ch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 scale=0.001 0.001 0.001
- link front_left_steering_link: geometry visual mesh filename=package://tadeocar_description/models/tadeocar_v1/meshes/su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 scale=1 1 1
- link front_left_wheel_link: geometry visual mesh filename=package://tadeocar_description/models/tadeocar_v1/meshes/wh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 scale=1 1 1
- link front_right_steering_link: geometry visual mesh filename=package://tadeocar_description/models/tadeocar_v1/meshes/su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 scale=1 1 1
- link front_right_wheel_link: geometry visual mesh filename=package://tadeocar_description/models/tadeocar_v1/meshes/wh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 scale=1 1 1
- link rear_left_steering_link: geometry visual mesh filename=package://tadeocar_description/models/tadeocar_v1/meshes/su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 scale=1 1 1
- link rear_left_wheel_link: geometry visual mesh filename=package://tadeocar_description/models/tadeocar_v1/meshes/wh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 scale=1 1 1
- link rear_right_steering_link: geometry visual mesh filename=package://tadeocar_description/models/tadeocar_v1/meshes/su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 scale=1 1 1
- link rear_right_wheel_link: geometry visual mesh filename=package://tadeocar_description/models/tadeocar_v1/meshes/wh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 scale=1 1 1

Commit message: vsalm

File: src/tadeocar_description/urdf/tadeocar.urdf (robot description, URDF)
Before this commit: robot tadeocar, 17 links, 16 joints
Links:
- removed link camera_left
- removed link camera_left_optical
- removed link camera_right
- removed link camera_right_optical
- removed link stereo_camera_base
- added link zed2i_camera_link; visual mesh filename=package://tadeocar_description/models/tadeocar_v1/meshes/se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 scale=0.001 0.001 0.001
- added link zed2i_imu_link
- added link zed2i_left_camera_optical_frame
- added link zed2i_right_camera_optical_frame
Joints:
- removed joint camera_left_joint
- removed joint camera_left_optical_joint
- removed joint camera_right_joint
- removed joint camera_right_optical_joint
- removed joint stereo_camera_base_joint
- added joint zed2i_camera_joint: type fixed, parent base_link, child zed2i_camera_link, origin xyz=0.55 0 0.40 rpy=0 0 0
- added joint zed2i_imu_joint: type fixed, parent zed2i_camera_link, child zed2i_imu_link, origin xyz=0 0 0 rpy=0 0 0
- added joint zed2i_left_optical_joint: type fixed, parent zed2i_camera_link, child zed2i_left_camera_optical_frame, origin xyz=0.005 0.06 0 rpy=-1.5708 0 -1.5708
- added joint zed2i_right_optical_joint: type fixed, parent zed2i_camera_link, child zed2i_right_camera_optical_frame, origin xyz=0.005 -0.06 0 rpy=-1.5708 0 -1.5708
