Commit message: Keep mass in the SDF alone, and give the plate and lamps their real one
The URDF is the robot's shape and carries no inertial tags, by design:
nothing simulates it. The tread plate and the upper chassis broke that
with inertials of their own, so the URDF described a 26 kg robot made
of two parts. Both are gone; the arc's mass derivation stays in its
comment.

In model.sdf the tread plate was 9.7 kg with box inertia. From its mesh
it is 1.098 m2 of 3 mm aluminium, 8.89 kg, plus two 0.785 m ribs of
40 x 20 x 2 mm tube, 0.95 kg: 9.84 kg, centre of mass at z 0.2645 in
base_link, inertia from the outline itself. The raised bars of the tread
pattern are not counted.

The lamps were 1.2 kg concentrated at base_link with 0.003 kg m2 about
every axis, as if they were one lump in the middle of the robot. They
are six lumps at the two ends: 0.25 kg per headlamp, 0.08 per indicator
and 0.27 per rear combination lamp, estimated, with nearly all of their
inertia about y and z (0.558 and 0.571 kg m2).

The model now weighs 126.6 kg, against 98.7 before the upper chassis,
the tread plate, the lamps and the second LiDAR.

File: src/tadeocar_description/urdf/tadeocar.urdf.xacro (robot description, xacro)
@@ -129,9 +129,4 @@
       <geometry><box size="1.34 0.76 ${plate_t}"/></geometry>
     </collision>
-    <inertial>
-      <origin xyz="-0.048 0 0.262" rpy="0 0 0"/>
-      <mass value="9.7"/>
-      <inertia ixx="0.5174" ixy="0" ixz="0" iyy="1.5844" iyz="0" izz="2.1016"/>
-    </inertial>
   </link>
   <joint name="deck_plate_joint" type="fixed">
@@ -154,7 +149,8 @@
        20 mm at each side. It stands on four corner foot plates bolted through
        the tread plate into the deck's rim.
-       Mass is not the mesh's: the mesh is solid, so its 12 071 cm3 is read as
-       9.66 m of tube and weighed as 50 x 25 x 1.5 mm steel, 16.4 kg. The
-       inertia is the mesh's own, scaled to that mass. -->
+       Its mass, which model.sdf carries like every other, is not the mesh's:
+       the mesh is solid, so its 12 071 cm3 is read as 9.66 m of tube and
+       weighed as 50 x 25 x 1.5 mm steel, 16.4 kg. The inertia is the mesh's
+       own, scaled to that mass. -->
   <link name="upper_chassis_link">
     <visual name="upper_chassis_visual">
@@ -188,9 +184,4 @@
     <xacro:arc_box name="arc_foot_rear_left"   x="-0.558" y="0.310"  z="0.015" sx="0.236" sy="0.156" sz="0.030"/>
     <xacro:arc_box name="arc_foot_rear_right"  x="-0.558" y="-0.310" z="0.015" sx="0.236" sy="0.156" sz="0.030"/>
-    <inertial>
-      <origin xyz="0.033 0 0.735" rpy="0 0 0"/>
-      <mass value="16.37"/>
-      <inertia ixx="4.784" ixy="0" ixz="0.1157" iyy="6.894" iyz="0" izz="5.132"/>
-    </inertial>
   </link>
   <joint name="upper_chassis_joint" type="fixed">
